Commit message: feat(mujoco): vendor upstream DiffBot and scale skin ×10
Replace simplified URDF with ros2_control_demos DiffBot sources plus a
plain expanded URDF at ~1 m footprint; keep mass/Izz for planar servos
and sync Godot puppet + spawn height.

Co-authored-by: Cursor <cursoragent@cursor.com>

File: mujoco/models/mechs/third_party/diffbot/diffbot.urdf (robot description, URDF)
Before this commit: robot diffbot, 5 links, 4 joints
Links:
- removed link caster
- removed link nose
- removed link wheel_left
- removed link wheel_right
- added link caster_frontal_wheel, mass 0.1; collision sphere radius=0.15; visual sphere radius=0.15
- added link caster_rear_wheel, mass 0.1; collision sphere radius=0.15; visual sphere radius=0.15
- added link left_wheel, mass 0.3; collision cylinder length=0.2 radius=0.15; visual cylinder length=0.2 radius=0.15
- added link right_wheel, mass 0.3; collision cylinder length=0.2 radius=0.15; visual cylinder length=0.2 radius=0.15
- link base_link: geometry collision box size=1.0 1.0 0.5; visual box size=1.0 1.0 0.5
Joints:
- removed joint caster_fixed
- removed joint nose_fixed
- removed joint wheel_left_joint
- removed joint wheel_right_joint
- added joint caster_frontal_wheel_joint: type fixed, parent base_link, child caster_frontal_wheel, origin xyz=0.35 0 -0.25 rpy=0 0 0
- added joint caster_rear_wheel_joint: type fixed, parent base_link, child caster_rear_wheel, origin xyz=-0.35 0 -0.25 rpy=0 0 0
- added joint left_wheel_joint: type continuous, parent base_link, child left_wheel, origin xyz=0 -0.5 -0.25 rpy=0 0 0, axis 0 1 0, limit effort=100 velocity=1.0
- added joint right_wheel_joint: type continuous, parent base_link, child right_wheel, origin xyz=0 0.5 -0.25 rpy=0 0 0, axis 0 1 0, limit effort=100 velocity=1.0
